File: ft234xd-breakout/ft234xd-breakout.sch (KiCad schematic (older format))
At the start: 18 parts, among them CON1 USB-MINI-B, P1 CONN_5, P2 CONN_5, U1 FT234XD

Commit message: fixed dfn12 pad spacing
Connections:
- wire segments 64 -> 82
Changed lines of the file:
@@
 Sheet 1 1
 Title ""
-Date "19 jan 2014"
+Date "17 feb 2014"
 Rev ""
 Comp ""
@@
 	2700 3050 3050 3050
 Wire Wire Line
-	2700 1900 2700 3050
+	2700 1900 2700 2050
+Wire Wire Line
+	2700 2050 2700 2350
+Wire Wire Line
+	2700 2350 2700 2500
+Wire Wire Line
+	2700 2500 2700 3050
 Wire Wire Line
 	2700 1900 2850 1900
@@
 	3150 2950 3050 2950
 Wire Wire Line
-	3050 2950 3050 3150
+	3050 2950 3050 3050
+Wire Wire Line
+	3050 3050 3050 3150
 Wire Wire Line
 	3050 3150 3200 3150
@@
 	3750 3150 3600 3150
 Wire Wire Line
-	3750 2950 3750 3150
+	3750 2950 3750 3050
+Wire Wire Line
+	3750 3050 3750 3150
 Wire Wire Line
 	3750 2950 3650 2950
 Wire Wire Line
-	3750 3050 4950 3050
+	3750 3050 4100 3050
+Wire Wire Line
+	4100 3050 4350 3050
+Wire Wire Line
+	4350 3050 4650 3050
+Wire Wire Line
+	4650 3050 4950 3050
 Wire Wire Line
 	4100 3050 4100 2500
@@
 Connection ~ 3750 3050
 Wire Wire Line
-	4350 2900 4350 3200
+	4350 2900 4350 3050
+Wire Wire Line
+	4350 3050 4350 3200
 Connection ~ 4100 3050
 Connection ~ 4350 3050
@@
 	4350 2500 4350 1900
 Wire Wire Line
-	3950 1900 4550 1900
+	3950 1900 4350 1900
+Wire Wire Line
+	4350 1900 4550 1900
 Wire Wire Line
 	4650 2500 4650 2200
 Wire Wire Line
-	3950 2200 5150 2200
-Wire Wire Line
-	3950 2050 5150 2050
+	3950 2200 4650 2200
+Wire Wire Line
+	4650 2200 5150 2200
+Wire Wire Line
+	3950 2050 4950 2050
+Wire Wire Line
+	4950 2050 5150 2050
 Wire Wire Line
 	4950 2050 4950 2500
@@
 Wire Wire Line
 	6250 5000 6900 5000
-Connection ~ 4350 1900
 Wire Wire Line
 	7300 2100 7200 2100
 Wire Wire Line
-	5750 4350 5750 5000
-Wire Wire Line
-	5750 4900 6900 4900
-Wire Wire Line
-	4050 4800 4050 5200
+	5750 4350 5750 4900
+Wire Wire Line
+	5750 4900 5750 5000
+Wire Wire Line
+	5750 4900 6050 4900
+Wire Wire Line
+	6050 4900 6900 4900
+Wire Wire Line
+	4050 4800 4050 5000
+Wire Wire Line
+	4050 5000 4050 5200
 Wire Wire Line
 	6750 4800 6900 4800
@@
 	4050 5800 4050 5600
 Wire Wire Line
-	5750 5400 5750 5800
+	5750 5400 5750 5500
+Wire Wire Line
+	5750 5500 5750 5800
 Connection ~ 5750 4900
 Wire Wire Line
@@
 	4850 5000 5050 5000
 Wire Wire Line
-	5050 4800 5050 5200
-Wire Wire Line
-	3850 5000 4250 5000
+	5050 4800 5050 5000
+Wire Wire Line
+	5050 5000 5050 5200
+Wire Wire Line
+	3850 5000 4050 5000
+Wire Wire Line
+	4050 5000 4250 5000
 Connection ~ 4050 5000
 Connection ~ 5050 5000
@@
 Wire Wire Line
 	3150 5000 3350 5000
+Connection ~ 4350 1900
 $EndSCHEMATC

Commit message: simplified and shrunk ft234xd board
Parts:
- removed C2: 0.1uF, ~, symbol C
- removed P1, P2: CONN_5, ~, symbol CONN_5
- added P1, P2: CONN_4, ~, symbol CONN_4
Connections:
- wire segments 82 -> 63
Changed lines of the file:
@@
-$EndComp
-$Comp
-L C C2
-U 1 1 52DA18FB
-P 4050 5400
-F 0 "C2" H 4050 5500 40  0000 L CNN
-F 1 "0.1uF" H 4056 5315 40  0000 L CNN
-F 2 "~" H 4088 5250 30  0000 C CNN
-F 3 "~" H 4050 5400 60  0000 C CNN
-	1    4050 5400
-	1    0    0    -1
-$EndComp
-$Comp
-L GND #PWR04
-U 1 1 52DA194E
-P 4050 5800
-F 0 "#PWR04" H 4050 5800 30  0001 C CNN
-F 1 "GND" H 4050 5730 30  0001 C CNN
-F 2 "" H 4050 5800 60  0000 C CNN
-F 3 "" H 4050 5800 60  0000 C CNN
-	1    4050 5800
-	1    0    0    -1
 $EndComp
 $Comp
@@
 $EndComp
 $Comp
-L GND #PWR05
+L GND #PWR04
 U 1 1 52DA1A18
 P 5750 5800
-F 0 "#PWR05" H 5750 5800 30  0001 C CNN
+F 0 "#PWR04" H 5750 5800 30  0001 C CNN
 F 1 "GND" H 5750 5730 30  0001 C CNN
 F 2 "" H 5750 5800 60  0000 C CNN
@@
 $EndComp
 $Comp
-L GND #PWR06
+L GND #PWR05
 U 1 1 52DA2324
 P 5050 5800
-F 0 "#PWR06" H 5050 5800 30  0001 C CNN
+F 0 "#PWR05" H 5050 5800 30  0001 C CNN
 F 1 "GND" H 5050 5730 30  0001 C CNN
 F 2 "" H 5050 5800 60  0000 C CNN
@@
 $EndComp
 $Comp
-L JUMPER JP1
-U 1 1 52DAA105
-P 4550 5000
-F 0 "JP1" H 4550 5150 60  0000 C CNN
-F 1 "JUMPER" H 4550 4920 40  0000 C CNN
-F 2 "~" H 4550 5000 60  0000 C CNN
-F 3 "~" H 4550 5000 60  0000 C CNN
-	1    4550 5000
-	1    0    0    -1
-$EndComp
-$Comp
-L CONN_5 P1
-U 1 1 52DAA2A9
-P 6800 2200
-F 0 "P1" V 6750 2200 50  0000 C CNN
-F 1 "CONN_5" V 6850 2200 50  0000 C CNN
-F 2 "~" H 6800 2200 60  0000 C CNN
-F 3 "~" H 6800 2200 60  0000 C CNN
-	1    6800 2200
-	-1   0    0    -1
-$EndComp
-$Comp
-L CONN_5 P2
-U 1 1 52DAA2B8
-P 8800 2200
-F 0 "P2" V 8750 2200 50  0000 C CNN
-F 1 "CONN_5" V 8850 2200 50  0000 C CNN
-F 2 "~" H 8800 2200 60  0000 C CNN
-F 3 "~" H 8800 2200 60  0000 C CNN
-	1    8800 2200
-	1    0    0    -1
-$EndComp
-$Comp
-L GND #PWR07
+L GND #PWR06
 U 1 1 52DAA6F1
 P 7750 2600
-F 0 "#PWR07" H 7750 2600 30  0001 C CNN
+F 0 "#PWR06" H 7750 2600 30  0001 C CNN
 F 1 "GND" H 7750 2530 30  0001 C CNN
 F 2 "" H 7750 2600 60  0000 C CNN
@@
 Text GLabel 6750 4600 0    60   Input ~ 0
 D-
-Text GLabel 8300 2000 0    60   Input ~ 0
+Text GLabel 7300 2300 2    60   Input ~ 0
 CBUS0
 Text GLabel 6750 5100 0    60   Input ~ 0
@@
 Text GLabel 7300 2200 2    60   Input ~ 0
 3V3OUT
-Text GLabel 7300 2300 2    60   Input ~ 0
-VCCIO
 Text GLabel 8650 4900 2    60   Input ~ 0
 VCCIO
 Text GLabel 5050 4800 1    60   Input ~ 0
 VCCIO
-Text GLabel 7300 2400 2    60   Input ~ 0
-RESET
 Text GLabel 7300 2100 2    60   Input ~ 0
 VBUS
@@
 Text GLabel 8650 5100 2    60   Input ~ 0
 TXD
+Text GLabel 8300 2200 0    60   Input ~ 0
+TXD
+Text GLabel 8300 2000 0    60   Input ~ 0
+RTS
 Text GLabel 8300 2300 0    60   Input ~ 0
-TXD
+RXD
 Text GLabel 8300 2100 0    60   Input ~ 0
-RTS
-Text GLabel 8300 2400 0    60   Input ~ 0
-RXD
-Text GLabel 8300 2200 0    60   Input ~ 0
 CTS
 NoConn ~ 3950 2350
@@
 	2700 3050 3050 3050
 Wire Wire Line
-	2700 1900 2700 2050
-Wire Wire Line
-	2700 2050 2700 2350
-Wire Wire Line
-	2700 2350 2700 2500
-Wire Wire Line
-	2700 2500 2700 3050
+	2700 1900 2700 3050
 Wire Wire Line
 	2700 1900 2850 1900
@@
 	3150 2950 3050 2950
 Wire Wire Line
-	3050 2950 3050 3050
-Wire Wire Line
-	3050 3050 3050 3150
+	3050 2950 3050 3150
 Wire Wire Line
 	3050 3150 3200 3150
@@
 	3750 3150 3600 3150
 Wire Wire Line
-	3750 2950 3750 3050
-Wire Wire Line
-	3750 3050 3750 3150
+	3750 2950 3750 3150
 Wire Wire Line
 	3750 2950 3650 2950
 Wire Wire Line
-	3750 3050 4100 3050
-Wire Wire Line
-	4100 3050 4350 3050
-Wire Wire Line
-	4350 3050 4650 3050
-Wire Wire Line
-	4650 3050 4950 3050
+	3750 3050 4950 3050
 Wire Wire Line
 	4100 3050 4100 2500
@@
 Connection ~ 3750 3050
 Wire Wire Line
-	4350 2900 4350 3050
-Wire Wire Line
-	4350 3050 4350 3200
+	4350 2900 4350 3200
 Connection ~ 4100 3050
 Connection ~ 4350 3050
@@
 	4350 2500 4350 1900
 Wire Wire Line
-	3950 1900 4350 1900
-Wire Wire Line
-	4350 1900 4550 1900
+	3950 1900 4550 1900
 Wire Wire Line
 	4650 2500 4650 2200
 Wire Wire Line
-	3950 2200 4650 2200
-Wire Wire Line
-	4650 2200 5150 2200
-Wire Wire Line
-	3950 2050 4950 2050
-Wire Wire Line
-	4950 2050 5150 2050
+	3950 2200 5150 2200
+Wire Wire Line
+	3950 2050 5150 2050
 Wire Wire Line
 	4950 2050 4950 2500
@@
 	7300 2100 7200 2100
 Wire Wire Line
-	5750 4350 5750 4900
-Wire Wire Line
-	5750 4900 5750 5000
-Wire Wire Line
-	5750 4900 6050 4900
-Wire Wire Line
-	6050 4900 6900 4900
-Wire Wire Line
-	4050 4800 4050 5000
-Wire Wire Line
-	4050 5000 4050 5200
+	5750 4350 5750 5000
+Wire Wire Line
+	5750 4900 6900 4900
 Wire Wire Line
 	6750 4800 6900 4800
 Wire Wire Line
-	4050 5800 4050 5600
-Wire Wire Line
-	5750 5400 5750 5500
-Wire Wire Line
-	5750 5500 5750 5800
+	5750 5400 5750 5800
 Connection ~ 5750 4900
 Wire Wire Line
@@
 	6750 5100 6900 5100
 Wire Wire Line
-	7300 2400 7200 2400
-Wire Wire Line
 	7300 2200 7200 2200
 Wire Wire Line
@@
 	6750 4700 6900 4700
 Wire Wire Line
-	4850 5000 5050 5000
-Wire Wire Line
-	5050 4800 5050 5000
-Wire Wire Line
-	5050 5000 5050 5200
-Wire Wire Line
-	3850 5000 4050 5000
-Wire Wire Line
-	4050 5000 4250 5000
-Connection ~ 4050 5000
+	3850 5000 5050 5000
+Wire Wire Line
+	5050 4800 5050 5200
 Connection ~ 5050 5000
 Wire Wire Line
-	8400 2200 8300 2200
-Wire Wire Line
-	8300 2400 8400 2400
-Wire Wire Line
 	8400 2100 8300 2100
 Wire Wire Line
@@
 Wire Wire Line
 	8400 2000 8300 2000
+Wire Wire Line
+	8300 2200 8400 2200
 Wire Wire Line
 	3150 5000 3350 5000
 Connection ~ 4350 1900
+$Comp
+L CONN_4 P2
+U 1 1 5301910A
+P 8750 2150
+F 0 "P2" V 8700 2150 50  0000 C CNN
+F 1 "CONN_4" V 8800 2150 50  0000 C CNN
+F 2 "~" H 8750 2150 60  0000 C CNN
+F 3 "~" H 8750 2150 60  0000 C CNN
+	1    8750 2150
+	1    0    0    -1
+$EndComp
+$Comp
+L CONN_4 P1
+U 1 1 53019119
+P 6850 2150
+F 0 "P1" V 6800 2150 50  0000 C CNN
+F 1 "CONN_4" V 6900 2150 50  0000 C CNN
+F 2 "~" H 6850 2150 60  0000 C CNN
+F 3 "~" H 6850 2150 60  0000 C CNN
+	1    6850 2150
+	-1   0    0    -1
+$EndComp
+Wire Wire Line
+	4050 4800 4050 5000
+Connection ~ 4050 5000
+$Comp
+L JUMPER JP1
+U 1 1 5301925E
+P 3600 5350
+F 0 "JP1" H 3600 5500 60  0000 C CNN
+F 1 "JUMPER" H 3600 5270 40  0000 C CNN
+F 2 "~" H 3600 5350 60  0000 C CNN
+F 3 "~" H 3600 5350 60  0000 C CNN
+	1    3600 5350
+	1    0    0    -1
+$EndComp
+Text GLabel 4050 5350 2    60   Input ~ 0
+CBUS0
+Wire Wire Line
+	4050 5350 3900 5350
+Wire Wire Line
+	3300 5350 3250 5350
+Wire Wire Line
+	3250 5350 3250 5000
+Connection ~ 3250 5000
 $EndSCHEMATC
