File: attiny20-bga-dip/attiny20-bga-dip.kicad_pcb (KiCad board)
At the start: 4 copper layers, 17.8 x 10.2 mm, 6 parts, among them P1 CONN_7, P2 CONN_7, P3 TC2030-IDC, U1 ATTINY20-CCU

Commit message: making attiny20 board OSH Park-friendly
Other:
- board text added: "GND"
- board text added: "PA0"
- board text added: "PA1"
- board text added: "PA2"
- board text added: "PA3"
- board text added: "PA4"
- board text added: "PA5"
- board text added: "PA6"
- board text added: "PA7"
- board text added: "PB0"
- board text added: "PB1"
- board text added: "PB2"
- board text added: "PB3"
- board text added: "Vcc"
Changed lines of the file:
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@@
     (area 192.110334 92.659999 212.167611 102.920001)
     (thickness 1.6)
-    (drawings 4)
+    (drawings 18)
     (tracks 107)
     (zones 0)
@@
   (page A3)
   (layers
-    (15 F.Cu signal)
+    (15 F.Cu signal hide)
     (2 Inner2.Cu signal hide)
     (1 Inner1.Cu signal hide)
-    (0 B.Cu signal)
-    (17 F.Adhes user)
-    (19 F.Paste user)
-    (21 F.SilkS user)
+    (0 B.Cu signal hide)
+    (17 F.Adhes user hide)
+    (19 F.Paste user hide)
+    (20 B.SilkS user)
+    (21 F.SilkS user hide)
     (23 F.Mask user)
     (28 Edge.Cuts user)
@@
     (visible_elements FFFFFFBF)
     (pcbplotparams
-      (layerselection 279478279)
+      (layerselection 280526855)
       (usegerberextensions true)
       (excludeedgelayer true)
@@
     )
   )
+  (gr_text PA5 (at 210.82 95.885 90) (layer B.SilkS)
+    (effects (font (size 0.508 0.508) (thickness 0.125)) (justify mirror))
+  )
+  (gr_text PA4 (at 208.28 95.885 90) (layer B.SilkS)
+    (effects (font (size 0.508 0.508) (thickness 0.125)) (justify mirror))
+  )
+  (gr_text PA3 (at 205.74 95.885 90) (layer B.SilkS)
+    (effects (font (size 0.508 0.508) (thickness 0.125)) (justify mirror))
+  )
+  (gr_text PA2 (at 203.2 95.885 90) (layer B.SilkS)
+    (effects (font (size 0.508 0.508) (thickness 0.125)) (justify mirror))
+  )
+  (gr_text PA1 (at 200.66 95.885 90) (layer B.SilkS)
+    (effects (font (size 0.508 0.508) (thickness 0.125)) (justify mirror))
+  )
+  (gr_text PA0 (at 198.12 95.885 90) (layer B.SilkS)
+    (effects (font (size 0.508 0.508) (thickness 0.125)) (justify mirror))
+  )
+  (gr_text GND (at 195.58 95.885 90) (layer B.SilkS)
+    (effects (font (size 0.508 0.508) (thickness 0.125)) (justify mirror))
+  )
+  (gr_text PA6 (at 210.82 99.695 90) (layer B.SilkS)
+    (effects (font (size 0.508 0.508) (thickness 0.127)) (justify mirror))
+  )
+  (gr_text PA7 (at 208.28 99.695 90) (layer B.SilkS)
+    (effects (font (size 0.508 0.508) (thickness 0.127)) (justify mirror))
+  )
+  (gr_text PB2 (at 205.74 99.695 90) (layer B.SilkS)
+    (effects (font (size 0.508 0.508) (thickness 0.127)) (justify mirror))
+  )
+  (gr_text PB3 (at 203.2 99.695 90) (layer B.SilkS)
+    (effects (font (size 0.508 0.508) (thickness 0.127)) (justify mirror))
+  )
+  (gr_text PB1 (at 200.66 99.695 90) (layer B.SilkS)
+    (effects (font (size 0.508 0.508) (thickness 0.127)) (justify mirror))
+  )
+  (gr_text "PB0\n" (at 198.12 99.695 90) (layer B.SilkS)
+    (effects (font (size 0.508 0.508) (thickness 0.127)) (justify mirror))
+  )
+  (gr_text Vcc (at 195.58 99.695 90) (layer B.SilkS)
+    (effects (font (size 0.508 0.508) (thickness 0.125)) (justify mirror))
+  )
   (gr_line (start 194.31 102.87) (end 194.31 92.71) (angle 90) (layer Edge.Cuts) (width 0.1))
