File: tpa2011d1-breakout/tpa2011d1-breakout.kicad_pcb (KiCad board)
At the start: 4 copper layers, 10.2 x 10.2 mm, 13 parts, among them P1 CONN_4, P2 CONN_4, U1 TPA2011D1

Commit message: fixing another board up to order
Other:
- board text added: "EN"
- board text added: "GND"
- board text added: "I+"
- board text added: "I-"
- board text added: "O+"
- board text added: "O-"
- board text added: "VDD"
Changed lines of the file:
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@@
     (links 24)
     (no_connects 0)
-    (area 212.89772 60.2234 223.774001 74.3966)
+    (area 213.105999 60.2234 223.86169 74.3966)
     (thickness 1.6)
-    (drawings 4)
+    (drawings 12)
     (tracks 64)
     (zones 0)
@@
   (page A3)
   (layers
-    (15 F.Cu signal)
+    (15 F.Cu signal hide)
     (2 Inner2.Cu signal hide)
     (1 Inner1.Cu signal hide)
-    (0 B.Cu signal)
-    (17 F.Adhes user)
+    (0 B.Cu signal hide)
     (19 F.Paste user)
+    (20 B.SilkS user hide)
     (21 F.SilkS user)
+    (22 B.Mask user)
     (23 F.Mask user)
     (28 Edge.Cuts user)
@@
     (visible_elements FFFFFFBF)
     (pcbplotparams
-      (layerselection 279478279)
+      (layerselection 284721159)
       (usegerberextensions true)
       (excludeedgelayer true)
@@
     (at 217.043 68.834 180)
     (attr smd)
-    (fp_text reference FB1 (at 0 0 270) (layer F.SilkS)
+    (fp_text reference FB1 (at 0 0 270) (layer F.SilkS) hide
       (effects (font (size 0.508 0.4572) (thickness 0.1143)))
     )
@@
     (at 219.837 68.834)
     (attr smd)
-    (fp_text reference FB2 (at 0 0 90) (layer F.SilkS)
+    (fp_text reference FB2 (at 0 0 90) (layer F.SilkS) hide
       (effects (font (size 0.508 0.4572) (thickness 0.1143)))
     )
@@
     (clearance 0.127)
     (attr smd)
-    (fp_text reference R2 (at 0 0 90) (layer F.SilkS)
+    (fp_text reference R2 (at 0 0 90) (layer F.SilkS) hide
       (effects (font (size 0.35052 0.3048) (thickness 0.07112)))
     )
@@
     (at 219.71 67.31 90)
     (attr smd)
-    (fp_text reference R1 (at 0 0 90) (layer F.SilkS)
+    (fp_text reference R1 (at 0 0 90) (layer F.SilkS) hide
       (effects (font (size 0.35052 0.3048) (thickness 0.07112)))
     )
@@
     (at 222.758 67.056 90)
     (descr "SMT capacitor, 0402")
-    (fp_text reference C2 (at 0 -0.4826 90) (layer F.SilkS)
+    (fp_text reference C2 (at 0 -0.4826 90) (layer F.SilkS) hide
       (effects (font (size 0.1524 0.1524) (thickness 0.03048)))
     )
@@
     (at 221.742 67.056 90)
     (descr "SMT capacitor, 0402")
-    (fp_text reference C1 (at 0 -0.4826 90) (layer F.SilkS)
+    (fp_text reference C1 (at 0 -0.4826 90) (layer F.SilkS) hide
       (effects (font (size 0.1524 0.1524) (thickness 0.03048)))
     )
@@
     (at 216.154 67.056 270)
     (descr "SMT capacitor, 0402")
-    (fp_text reference C4 (at 0 0 360) (layer F.SilkS)
+    (fp_text reference C4 (at 0 0 360) (layer F.SilkS) hide
       (effects (font (size 0.1524 0.1524) (thickness 0.03048)))
     )
@@
     (at 220.726 67.056 270)
     (descr "SMT capacitor, 0402")
-    (fp_text reference C5 (at 0 0 360) (layer F.SilkS)
+    (fp_text reference C5 (at 0 0 360) (layer F.SilkS) hide
       (effects (font (size 0.1524 0.1524) (thickness 0.03048)))
     )
@@
     (at 214.63 67.31 90)
     (descr "SMT capacitor, 1206")
-    (fp_text reference C6 (at 0.0254 -1.2954 90) (layer F.SilkS)
+    (fp_text reference C6 (at 0 -0.762 90) (layer F.SilkS) hide
       (effects (font (size 0.50038 0.50038) (thickness 0.11938)))
     )
@@
     (at 218.44 66.04 180)
     (descr "SMT capacitor, 0402")
-    (fp_text reference C3 (at 0 -0.4826 180) (layer F.SilkS)
+    (fp_text reference C3 (at 0 -0.4826 180) (layer F.SilkS) hide
       (effects (font (size 0.1524 0.1524) (thickness 0.03048)))
     )
@@
     )
   )
+  (gr_text VDD (at 214.63 65.024 90) (layer B.SilkS)
+    (effects (font (size 0.508 0.508) (thickness 0.127)) (justify left mirror))
+  )
+  (gr_text I+ (at 217.17 65.024 90) (layer B.SilkS)
+    (effects (font (size 0.508 0.508) (thickness 0.127)) (justify left mirror))
+  )
+  (gr_text "I-\n" (at 219.71 65.024 90) (layer B.SilkS)
+    (effects (font (size 0.508 0.508) (thickness 0.127)) (justify left mirror))
+  )
+  (gr_text GND (at 222.25 65.024 90) (layer B.SilkS)
+    (effects (font (size 0.508 0.508) (thickness 0.127)) (justify left mirror))
+  )
+  (gr_text GND (at 222.25 69.596 90) (layer B.SilkS)
+    (effects (font (size 0.508 0.508) (thickness 0.127)) (justify right mirror))
+  )
+  (gr_text O- (at 219.71 69.596 90) (layer B.SilkS)
+    (effects (font (size 0.508 0.508) (thickness 0.127)) (justify right mirror))
+  )
+  (gr_text O+ (at 217.17 69.596 90) (layer B.SilkS)
+    (effects (font (size 0.508 0.508) (thickness 0.127)) (justify right mirror))
+  )
+  (gr_text EN (at 214.63 69.596 90) (layer B.SilkS)
+    (effects (font (size 0.508 0.508) (thickness 0.127)) (justify right mirror))
+  )
   (gr_line (start 223.52 72.39) (end 213.36 72.39) (angle 90) (layer Edge.Cuts) (width 0.1))
