File: max34406-dip-module/max34406-dip-module.kicad_pcb (KiCad board)
At the start: 4 copper layers, 27.9 x 10.2 mm, 12 parts, among them P1 CONN_11, P2 CONN_11, U1 MAX34406

Commit message: grr... "bottom silk screen; image [can't be blank]"
Other:
- board text added: "MAX34406 breakout v0"
Changed lines of the file:
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@@
     (area 184.762096 118.12524 214.017904 131.191001)
     (thickness 1.6)
-    (drawings 4)
+    (drawings 5)
     (tracks 191)
     (zones 0)
@@
     (19 F.Paste user)
     (20 B.SilkS user)
-    (21 F.SilkS user hide)
+    (21 F.SilkS user)
     (22 B.Mask user)
     (23 F.Mask user)
@@
     (visible_elements FFFFFFBF)
     (pcbplotparams
-      (layerselection 284983303)
+      (layerselection 3145728)
       (usegerberextensions true)
       (excludeedgelayer true)
@@
     (uvia_drill 0.127)
   )
+  (module SIL-11 (layer F.Cu)
+    (at 200.66 129.54)
+    (descr "Connecteur 12 pins")
+    (tags "CONN DEV")
+    (fp_text reference P2 (at -7.62 -2.54) (layer F.SilkS) hide
+      (effects (font (size 1.72974 1.08712) (thickness 0.27178)))
+    )
+    (fp_text value CONN_11 (at 7.62 -2.54) (layer F.SilkS) hide
+      (effects (font (size 1.524 1.016) (thickness 0.254)))
+    )
+    (fp_line (start -12.7 1.27) (end 12.7 1.27) (layer F.SilkS) (width 0.254))
+    (fp_line (start 12.7 1.27) (end 12.7 -1.27) (layer F.SilkS) (width 0.254))
+    (fp_line (start 12.7 -1.27) (end -12.7 -1.27) (layer F.SilkS) (width 0.254))
+    (fp_line (start -15.24 1.27) (end -15.24 -1.27) (layer F.SilkS) (width 0.254))
+    (fp_line (start -15.24 -1.27) (end -12.7 -1.27) (layer F.SilkS) (width 0.254))
+    (fp_line (start -12.7 1.27) (end -15.24 1.27) (layer F.SilkS) (width 0.254))
+    (pad 1 thru_hole circle (at -13.97 0) (size 1.397 1.397) (drill 0.8128)
+      (layers *.Cu *.Mask F.SilkS)
+      (net 17 /OUT1)
+    )
+    (pad 2 thru_hole circle (at -11.43 0) (size 1.397 1.397) (drill 0.8128)
+      (layers *.Cu *.Mask F.SilkS)
+      (net 12 /OC1)
+    )
+    (pad 3 thru_hole circle (at -8.89 0) (size 1.397 1.397) (drill 0.8128)
+      (layers *.Cu *.Mask F.SilkS)
+      (net 18 /OUT2)
+    )
+    (pad 4 thru_hole circle (at -6.35 0) (size 1.397 1.397) (drill 0.8128)
+      (layers *.Cu *.Mask F.SilkS)
+      (net 13 /OC2)
+    )
+    (pad 5 thru_hole circle (at -3.81 0) (size 1.397 1.397) (drill 0.8128)
+      (layers *.Cu *.Mask F.SilkS)
+      (net 3 /GND)
+    )
+    (pad 6 thru_hole circle (at -1.27 0) (size 1.397 1.397) (drill 0.8128)
+      (layers *.Cu *.Mask F.SilkS)
+      (net 22 /VDD)
+    )
+    (pad 7 thru_hole circle (at 1.27 0) (size 1.397 1.397) (drill 0.8128)
+      (layers *.Cu *.Mask F.SilkS)
+      (net 16 /OC_PU)
+    )
+    (pad 8 thru_hole circle (at 3.81 0) (size 1.397 1.397) (drill 0.8128)
+      (layers *.Cu *.Mask F.SilkS)
+      (net 19 /OUT3)
+    )
+    (pad 9 thru_hole circle (at 6.35 0) (size 1.397 1.397) (drill 0.8128)
+      (layers *.Cu *.Mask F.SilkS)
+      (net 14 /OC3)
+    )
+    (pad 10 thru_hole circle (at 8.89 0) (size 1.397 1.397) (drill 0.8128)
+      (layers *.Cu *.Mask F.SilkS)
+      (net 20 /OUT4)
+    )
+    (pad 11 thru_hole circle (at 11.43 0) (size 1.397 1.397) (drill 0.8128)
+      (layers *.Cu *.Mask F.SilkS)
+      (net 15 /OC4)
+    )
+    (model pin_array\pins_array_12x1.wrl
+      (at (xyz 0 0 0))
+      (scale (xyz 1 1 1))
+      (rotate (xyz 0 0 0))
+    )
+  )
   (module QFN24 (layer F.Cu)
     (at 199.39 125.73)
@@
     )
   )
-  (module SIL-11 (layer F.Cu)
-    (at 200.66 129.54)
-    (descr "Connecteur 12 pins")
-    (tags "CONN DEV")
-    (fp_text reference P2 (at -7.62 -2.54) (layer F.SilkS) hide
-      (effects (font (size 1.72974 1.08712) (thickness 0.27178)))
-    )
-    (fp_text value CONN_11 (at 7.62 -2.54) (layer F.SilkS) hide
-      (effects (font (size 1.524 1.016) (thickness 0.254)))
-    )
-    (fp_line (start -12.7 1.27) (end 12.7 1.27) (layer F.SilkS) (width 0.254))
-    (fp_line (start 12.7 1.27) (end 12.7 -1.27) (layer F.SilkS) (width 0.254))
-    (fp_line (start 12.7 -1.27) (end -12.7 -1.27) (layer F.SilkS) (width 0.254))
-    (fp_line (start -15.24 1.27) (end -15.24 -1.27) (layer F.SilkS) (width 0.254))
-    (fp_line (start -15.24 -1.27) (end -12.7 -1.27) (layer F.SilkS) (width 0.254))
-    (fp_line (start -12.7 -1.27) (end -12.7 1.27) (layer F.SilkS) (width 0.254))
-    (fp_line (start -12.7 1.27) (end -15.24 1.27) (layer F.SilkS) (width 0.254))
-    (pad 1 thru_hole circle (at -13.97 0) (size 1.397 1.397) (drill 0.8128)
-      (layers *.Cu *.Mask F.SilkS)
-      (net 17 /OUT1)
-    )
-    (pad 2 thru_hole circle (at -11.43 0) (size 1.397 1.397) (drill 0.8128)
-      (layers *.Cu *.Mask F.SilkS)
-      (net 12 /OC1)
-    )
-    (pad 3 thru_hole circle (at -8.89 0) (size 1.397 1.397) (drill 0.8128)
-      (layers *.Cu *.Mask F.SilkS)
-      (net 18 /OUT2)
-    )
-    (pad 4 thru_hole circle (at -6.35 0) (size 1.397 1.397) (drill 0.8128)
-      (layers *.Cu *.Mask F.SilkS)
-      (net 13 /OC2)
-    )
-    (pad 5 thru_hole circle (at -3.81 0) (size 1.397 1.397) (drill 0.8128)
-      (layers *.Cu *.Mask F.SilkS)
-      (net 3 /GND)
-    )
-    (pad 6 thru_hole circle (at -1.27 0) (size 1.397 1.397) (drill 0.8128)
-      (layers *.Cu *.Mask F.SilkS)
-      (net 22 /VDD)
-    )
-    (pad 7 thru_hole circle (at 1.27 0) (size 1.397 1.397) (drill 0.8128)
-      (layers *.Cu *.Mask F.SilkS)
-      (net 16 /OC_PU)
-    )
-    (pad 8 thru_hole circle (at 3.81 0) (size 1.397 1.397) (drill 0.8128)
-      (layers *.Cu *.Mask F.SilkS)
-      (net 19 /OUT3)
-    )
-    (pad 9 thru_hole circle (at 6.35 0) (size 1.397 1.397) (drill 0.8128)
-      (layers *.Cu *.Mask F.SilkS)
-      (net 14 /OC3)
-    )
-    (pad 10 thru_hole circle (at 8.89 0) (size 1.397 1.397) (drill 0.8128)
-      (layers *.Cu *.Mask F.SilkS)
-      (net 20 /OUT4)
-    )
-    (pad 11 thru_hole circle (at 11.43 0) (size 1.397 1.397) (drill 0.8128)
-      (layers *.Cu *.Mask F.SilkS)
-      (net 15 /OC4)
-    )
-    (model pin_array\pins_array_12x1.wrl
-      (at (xyz 0 0 0))
-      (scale (xyz 1 1 1))
-      (rotate (xyz 0 0 0))
-    )
-  )
   (module SM0402_r (layer F.Cu)
     (at 211.455 127.635)
@@
     )
   )
+  (gr_text "MAX34406 breakout v0" (at 206.375 127.635) (layer B.SilkS)
+    (effects (font (size 0.762 0.762) (thickness 0.1905)) (justify mirror))
+  )
   (gr_line (start 185.42 130.81) (end 185.42 120.65) (angle 90) (layer Edge.Cuts) (width 0.1))
