File: pdi-dongle/pdi-dongle.sch (KiCad schematic (older format))
At the start: 6 parts, among them P101 CONN_6, P102 CONN_10

Commit message: new version of the PDI adapter board
Connections:
- net PDI_D: now also P102.3 (P3); no longer P102.4 (P4)
- net VREF: now also P102.4 (P4); no longer P102.3 (P3)
Changed lines of the file:
@@
 Sheet 1 1
 Title ""
-Date "27 may 2014"
+Date "5 aug 2014"
 Rev ""
 Comp ""
@@
 Wire Wire Line
 	7900 3700 7600 3700
+Text Label 8200 3300 0    60   ~ 0
+VREF
 Text Label 8200 3200 0    60   ~ 0
-VREF
-Text Label 8200 3300 0    60   ~ 0
 PDI_D
 Text Label 8200 3500 0    60   ~ 0
