File: microSD-breakout/microSD-breakout.kicad_pcb (KiCad board)
At the start: 2 copper layers, 20.3 x 15.9 mm, 11 parts, among them P1 CONN_5, P2 CONN_5, U1 MIC5504-3.3, U2 MICROSD_JAE_ST11-H

Commit message: changed some stuff.  a long time ago, so i don't remember what.
Parts:
- U2: footprint MICROSD_JAE_ST11-H -> mokus:MICROSD_JAE_ST11-H
- moved R3 10.3 mm to (273.5, 104.5), turned to 0 degrees
- moved R1 6.98 mm to (278.0, 104.1), turned to 90 degrees
- moved R2 6.73 mm to (278.0, 105.0), turned to 270 degrees
- moved C3 0.19 mm to (280.0, 110.4)
- moved TP1 0.08 mm to (287.0, 103.2)
Routing:
- net /VIN: track 28.6 -> 15.0 mm, vias 3 -> 1
- net /EN: track 17.6 -> 5.17 mm, vias 2 -> 0
- net /DSW: track 18.0 -> 29.0 mm
- net /GND: track 14.9 -> 7.18 mm
