File: microSD-breakout/microSD-breakout.kicad_pcb (KiCad board)
At the start: 2 copper layers, 20.3 x 15.9 mm, 11 parts, among them P1 CONN_5, P2 CONN_5, U1 MIC5504-3.3, U2 MICROSD_JAE_ST11-H

Commit message: changed some other stuff...  this will probably conflict
Routing:
- net /DSW: track 18.0 -> 16.9 mm
- net /VIN: track 28.6 -> 28.0 mm
