File: microSD-breakout/microSD-breakout.sch (KiCad schematic (older format))
At the start: 11 parts, among them P1 CONN_5, P2 CONN_5, U1 MIC5504-3.3YM5 TR, U2 MICROSD_JAE_ST11-H

Commit message: changed some stuff.  a long time ago, so i don't remember what.
Changed lines of the file:
@@
 LIBS:parts
 LIBS:microSD-breakout-cache
-EELAYER 27 0
+EELAYER 25 0
 EELAYER END
 $Descr A4 11693 8268
@@
 	5400 1300 5400 1400
 Connection ~ 5400 1400
-Text Notes 3300 2800 0    60   ~ 0
+Text Notes 3350 3000 0    60   ~ 0
 DSW is open when card is present, pulled to ground when card is absent\nSo we pull that up to VIN and (optionally) use it to enable the regulator.\nAlternately we can pull DSW up to the 3V3 rail for use by the MCU
 Text Label 3400 1900 0    60   ~ 0
